File: hardware/eletricalSchema/v1/thereef/thereef.kicad_sch (KiCad schematic)
At the start: 6 parts, among them J1 Output terminal, K1 SANYOU_SRD_Form_C, K2 SANYOU_SRD_Form_C, U1 Olimex_MOD-WIFI-ESP8266-DEV

Commit message: chore: remove unnecessary set high pin value
Parts:
- removed R2: 270K, symbol Device:R
Connections:
- net GND: now also J1.4 (Pin_4)
- net SB Input: now also K1.2
- net VCC (5V): no longer J1.4 (Pin_4)
Changed lines of the file:
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@@
+	)
+	(junction
+		(at 201.93 67.31)
+		(diameter 0)
+		(color 0 0 0 0)
 	)
 	(junction
@@
 	(wire
 		(pts
+			(xy 201.93 68.58) (xy 201.93 67.31)
+		)
+		(stroke
+			(width 0)
+			(type default)
+		)
+	)
+	(wire
+		(pts
 			(xy 185.42 57.15) (xy 185.42 59.69)
 		)
@@
 	(wire
 		(pts
+			(xy 201.93 67.31) (xy 201.93 66.04)
+		)
+		(stroke
+			(width 0)
+			(type default)
+		)
+	)
+	(wire
+		(pts
 			(xy 185.42 59.69) (xy 185.42 60.96)
 		)
@@
 	(wire
 		(pts
+			(xy 199.39 67.31) (xy 201.93 67.31)
+		)
+		(stroke
+			(width 0)
+			(type default)
+		)
+	)
+	(wire
+		(pts
 			(xy 181.61 114.3) (xy 207.01 114.3)
 		)
@@
 	(wire
 		(pts
-			(xy 193.04 68.58) (xy 208.28 68.58)
-		)
-		(stroke
-			(width 0)
-			(type default)
-		)
-	)
-	(wire
-		(pts
 			(xy 201.93 73.66) (xy 208.28 73.66)
 		)
@@
 	(wire
 		(pts
-			(xy 175.26 82.55) (xy 175.26 97.79)
+			(xy 208.28 68.58) (xy 201.93 68.58)
 		)
 		(stroke
@@
 	(wire
 		(pts
-			(xy 175.26 73.66) (xy 175.26 74.93)
+			(xy 175.26 73.66) (xy 175.26 97.79)
 		)
 		(stroke
@@
 	)
 	(symbol
-		(lib_id "Device:R")
-		(at 175.26 78.74 0)
-		(unit 1)
-		(exclude_from_sim no)
-		(in_bom yes)
-		(on_board yes)
-		(dnp no)
-		(property "Reference" "R2"
-			(at 172.212 75.946 90)
-			(effects
-				(font
-					(size 1.27 1.27)
-				)
-			)
-		)
-		(property "Value" "270K"
-			(at 178.054 78.994 90)
-			(effects
-				(font
-					(size 1.27 1.27)
-				)
-			)
-		)
-		(property "Footprint" ""
-			(at 173.482 78.74 90)
-			(effects
-				(font
-					(size 1.27 1.27)
-				)
-				(hide yes)
-			)
-		)
-		(property "Datasheet" "~"
-			(at 175.26 78.74 0)
-			(effects
-				(font
-					(size 1.27 1.27)
-				)
-				(hide yes)
-			)
-		)
-		(property "Description" "Resistor"
-			(at 175.26 78.74 0)
-			(effects
-				(font
-					(size 1.27 1.27)
-				)
-				(hide yes)
-			)
-		)
-		(pin "2"
-		)
-		(pin "1"
-		)
-		(instances
-			(project ""
-				(path "/b8fdac2d-f99e-46e5-973e-bafd98e5703f"
-					(reference "R2")
-					(unit 1)
-				)
-			)
-		)
-	)
-	(symbol
 		(lib_id "power:GND")
 		(at 170.18 113.03 90)
@@
 	)
 	(symbol
-		(lib_id "power:VCC")
-		(at 193.04 68.58 90)
-		(unit 1)
-		(exclude_from_sim no)
-		(in_bom yes)
-		(on_board yes)
-		(dnp no)
-		(property "Reference" "#PWR04"
-			(at 196.85 68.58 0)
-			(effects
-				(font
-					(size 1.27 1.27)
-				)
-				(hide yes)
-			)
-		)
-		(property "Value" "VCC (5V)"
-			(at 194.564 67.056 90)
-			(effects
-				(font
-					(size 1.27 1.27)
-				)
-			)
-		)
-		(property "Footprint" ""
-			(at 193.04 68.58 0)
-			(effects
-				(font
-					(size 1.27 1.27)
-				)
-				(hide yes)
-			)
-		)
-		(property "Datasheet" ""
-			(at 193.04 68.58 0)
-			(effects
-				(font
-					(size 1.27 1.27)
-				)
-				(hide yes)
-			)
-		)
-		(property "Description" "Power symbol creates a global label with name \"VCC\""
-			(at 193.04 68.58 0)
-			(effects
-				(font
-					(size 1.27 1.27)
-				)
-				(hide yes)
-			)
-		)
-		(pin "1"
-		)
-		(instances
-			(project ""
-				(path "/b8fdac2d-f99e-46e5-973e-bafd98e5703f"
-					(reference "#PWR04")
-					(unit 1)
-				)
-			)
-		)
-	)
-	(symbol
 		(lib_id "power:GND")
-		(at 201.93 66.04 270)
+		(at 199.39 67.31 270)
 		(unit 1)
 		(exclude_from_sim no)
@@
 		(dnp no)
 		(property "Reference" "#PWR02"
-			(at 195.58 66.04 0)
+			(at 193.04 67.31 0)
 			(effects
 				(font
@@
 		)
 		(property "Value" "GND"
-			(at 204.724 65.024 90)
+			(at 198.628 65.278 90)
 			(effects
 				(font
@@
 		)
 		(property "Footprint" ""
-			(at 201.93 66.04 0)
+			(at 199.39 67.31 0)
 			(effects
 				(font
@@
 		)
 		(property "Datasheet" ""
-			(at 201.93 66.04 0)
+			(at 199.39 67.31 0)
 			(effects
 				(font
@@
 		)
 		(property "Description" "Power symbol creates a global label with name \"GND\" , ground"
-			(at 201.93 66.04 0)
-			(effects
-				(font
+			(at 199.39 67.31 0)
+			(effects
+				(font
